File: batty-classic/pbc/batty.kicad_pcb (KiCad board)
At the start: 2 copper layers, 137.4 x 95.2 mm, 102 parts, among them J1 MJ-4PP-9, J2 OLED, J3 LED, P1 i2c-pin, P2 i2c-pin, SW1 SW_PUSH, SW10 SW_PUSH, SW11 SW_PUSH, SW12 SW_PUSH, SW13 SW_PUSH, SW14 SW_PUSH, SW15 SW_PUSH, SW16 SW_PUSH, SW17 SW_PUSH, SW18 SW_PUSH, SW19 SW_PUSH, SW2 SW_PUSH, SW20 SW_PUSH, SW21 SW_PUSH, SW22 SW_PUSH, SW23 SW_PUSH, SW3 SW_PUSH, SW4 SW_PUSH, SW5 SW_PUSH, SW6 SW_PUSH, SW7 SW_PUSH, SW8 SW_PUSH, SW9 SW_PUSH, U1 ProMicro

Commit message: add batty-classic
Parts:
- removed the G*** at (184.0, 78.0)
- removed the G*** at (184.7, 78.0)
- added G***: logo, batty:logo_background, F.Cu at (184.3, 83.3)
- added G***: logo, batty:logo, F.Cu at (185.0, 70.4)
- moved L29 2.27 mm to (182.5, 124.7)
- moved SW23 2.18 mm to (187.2, 127.6)
- moved ? 1.72 mm to (191.7, 116.2)
- moved ? 1.24 mm to (178.4, 108.8)
- moved J1 0.93 mm to (194.8, 109.7)
- moved JP1 0.93 mm to (181.2, 105.8)
- moved JP2 0.93 mm to (188.9, 94.2)
- moved JP3 0.93 mm to (186.4, 94.2)
- moved JP4 0.93 mm to (183.9, 94.2)
- moved JP5 0.93 mm to (181.4, 94.2)
- moved JP6 0.93 mm to (188.9, 94.2)
- moved JP7 0.93 mm to (186.4, 94.2)
- moved JP8 0.93 mm to (183.9, 94.2)
- moved JP9 0.93 mm to (181.4, 94.2)
- moved P1 0.93 mm to (181.1, 101.0)
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Routing:
- net Net-(L27-Pad3): track 48.8 -> 54.9 mm
- net col6: track 83.7 -> 87.4 mm, vias 7 -> 4
- net LED: track 86.6 -> 89.9 mm
- net GND: track 921.1 -> 923.9 mm
- net col3: track 230.1 -> 231.5 mm
- net row1: track 174.9 -> 176.2 mm
- net col2: track 202.4 -> 203.5 mm
- net col4: track 199.2 -> 200.4 mm
- net col1: track 217.7 -> 216.7 mm
- net row2: track 199.3 -> 200.4 mm
- net row3: track 201.6 -> 202.5 mm
- net col0: track 274.0 -> 273.1 mm
- net col5: track 202.2 -> 202.9 mm
- net VCC: track 831.7 -> 832.4 mm
- net reset: track 42.8 -> 42.2 mm
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Other:
- board size 137.4 x 95.2 mm -> 138.5 x 95.2 mm
- board text added: "Batty v0.2 PCB modified by hirakiuc"
- board text removed: "Batty v0.1 PCB Designed by hirakiuc"
